File: truckpad/truckpad.kicad_pcb (KiCad board)
At the start: 2 copper layers, 98 x 42.3 mm, 11 parts, among them J1 OLED-128x32, SW1 SW_Push, SW2 SW_Push, SW3 SW_Push, SW4 SW_Push, SW5 RotaryEncoder_Switch, U1 XIAO-RP2040-DIP

Commit message: update
Parts:
- renumbered Modifier_D1 to Modifier, Status_D1 to Status
